File: KiCAD/SZG-SDI-12G-Fire/SZG-SDI-12G-Fire.kicad_sch (KiCad schematic)
At the start: 28 parts, among them J1 SYZYGY_TXR-4, U15 LP5907MFX-2.5/NOPB, U4 513FCA000270AAG

Commit message: Initial version: Rev.A
Minor schematic tweaks for routing and to address SDI Rx/Tx power rails
PCB fully placed and routed
Added README/CHANGES files
Added CERN-OHL-P v2 license file

Signed-off-by: Charles Steinkuehler <charles@steinkuehler.net>
Connections:
- net CLK_FS: now also J1.17 (S2); no longer J1.19 (S4)
- net CLK_OE: now also J1.19 (S4); no longer J1.17 (S2)
- net CS_n: now also J1.16 (S1); no longer J1.20 (S5)
- net SCLK: now also J1.20 (S5); no longer J1.16 (S1)
Changed lines of the file:
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@@
     (company "Opal Kelly Incorporated")
   )
+  (junction (at 238.76 134.62) (diameter 0) (color 0 0 0 0)
+  )
   (junction (at 62.23 160.02) (diameter 0) (color 0 0 0 0)
   )
@@
   )
   (junction (at 62.23 152.4) (diameter 0) (color 0 0 0 0)
+  )
+  (junction (at 238.76 124.46) (diameter 0) (color 0 0 0 0)
   )
   (junction (at 138.43 186.69) (diameter 0) (color 0 0 0 0)
@@
     (stroke (width 0) (type default))
   )
+  (wire (pts (xy 238.76 121.92) (xy 238.76 124.46))
+    (stroke (width 0) (type default))
+  )
   (wire (pts (xy 62.23 167.64) (xy 62.23 175.26))
     (stroke (width 0) (type default))
@@
   )
   (wire (pts (xy 208.28 58.42) (xy 223.52 58.42))
+    (stroke (width 0) (type default))
+  )
+  (wire (pts (xy 238.76 134.62) (xy 238.76 137.16))
     (stroke (width 0) (type default))
   )
@@
     (effects (font (size 1.27 1.27)) (justify left bottom))
   )
-  (label "CLK_OE" (at 39.37 82.55 0) (fields_autoplaced)
+  (label "CLK_OE" (at 39.37 85.09 0) (fields_autoplaced)
     (effects (font (size 1.27 1.27)) (justify left bottom))
   )
@@
     (effects (font (size 1.27 1.27)) (justify left bottom))
   )
-  (label "SCLK" (at 82.55 77.47 0) (fields_autoplaced)
+  (label "SCLK" (at 82.55 85.09 0) (fields_autoplaced)
     (effects (font (size 1.27 1.27)) (justify left bottom))
   )
@@
     (effects (font (size 1.27 1.27)) (justify left bottom))
   )
-  (label "CLK_FS" (at 39.37 85.09 0) (fields_autoplaced)
+  (label "CLK_FS" (at 39.37 82.55 0) (fields_autoplaced)
     (effects (font (size 1.27 1.27)) (justify left bottom))
   )
@@
     (effects (font (size 1.27 1.27)) (justify left bottom))
   )
-  (label "CS_n" (at 82.55 85.09 0) (fields_autoplaced)
+  (label "CS_n" (at 82.55 77.47 0) (fields_autoplaced)
     (effects (font (size 1.27 1.27)) (justify left bottom))
   )
@@
     (effects (font (size 1.27 1.27)) (justify left bottom))
   )
+  (netclass_flag "" (length 2.54) (shape round) (at 238.76 121.92 0) (fields_autoplaced)
+    (effects (font (size 1.27 1.27)) (justify left bottom))
+    (property "Netclass" "100R" (at 239.3696 119.38 0)
+      (effects (font (size 1.27 1.27) italic) (justify left))
+    )
+  )
+  (netclass_flag "" (length 2.54) (shape round) (at 238.76 137.16 180) (fields_autoplaced)
+    (effects (font (size 1.27 1.27)) (justify right bottom))
+    (property "Netclass" "100R" (at 239.3696 139.7 0)
+      (effects (font (size 1.27 1.27) italic) (justify left))
+    )
+  )
+  (netclass_flag "" (length 2.54) (shape round) (at 264.16 134.62 180) (fields_autoplaced)
+    (effects (font (size 1.27 1.27)) (justify right bottom))
+    (property "Netclass" "100R" (at 264.7696 137.16 0)
+      (effects (font (size 1.27 1.27) italic) (justify left))
+    )
+  )
+  (netclass_flag "" (length 2.54) (shape round) (at 264.16 124.46 180) (fields_autoplaced)
+    (effects (font (size 1.27 1.27)) (justify right bottom))
+    (property "Netclass" "100R" (at 264.7696 127 0)
+      (effects (font (size 1.27 1.27) italic) (justify left))
+    )
+  )
   (symbol (lib_id "power:GND") (at 66.04 134.62 0) (unit 1)

Commit message: Update with part numbers
Add manufacturer part numbers as ordered from DigiKey
Add stitching vias on PCB for SDI 75 ohm striplines

Signed-off-by: Charles Steinkuehler <charles@steinkuehler.net>
Parts:
- C33, C34: Manufacturer (none) -> Murata; Manufacturer_PN (none) -> GRM155R70J105KA12J
- R1: Manufacturer (none) -> Yageo; Manufacturer_PN (none) -> RC0402FR-0710KL
- R10, R11, R12, R5, R6, R7, R8, R9: Manufacturer (none) -> Yageo; Manufacturer_PN (none) -> RC0402FR-070RL
Changed lines of the file:
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@@
+      (effects (font (size 1.27 1.27)) hide)
+    )
+    (property "Manufacturer" "Yageo" (at 102.87 46.99 0)
+      (effects (font (size 1.27 1.27)) hide)
+    )
+    (property "Manufacturer_PN" "RC0402FR-0710KL" (at 102.87 46.99 0)
       (effects (font (size 1.27 1.27)) hide)
     )
@@
       (effects (font (size 1.27 1.27)) hide)
     )
+    (property "Manufacturer_PN" "RC0402FR-070RL" (at 55.88 175.26 0)
+      (effects (font (size 1.27 1.27)) hide)
+    )
+    (property "Manufacturer" "Yageo" (at 55.88 175.26 0)
+      (effects (font (size 1.27 1.27)) hide)
+    )
     (pin "1")
     (pin "2")
@@
       (effects (font (size 1.27 1.27)) hide)
     )
+    (property "Manufacturer" "Murata" (at 158.75 146.05 0)
+      (effects (font (size 1.27 1.27)) hide)
+    )
+    (property "Manufacturer_PN" "GRM155R70J105KA12J" (at 158.75 146.05 0)
+      (effects (font (size 1.27 1.27)) hide)
+    )
     (pin "1")
     (pin "2")
@@
       (effects (font (size 1.27 1.27)) hide)
     )
+    (property "Manufacturer" "Murata" (at 146.05 146.05 0)
+      (effects (font (size 1.27 1.27)) hide)
+    )
+    (property "Manufacturer_PN" "GRM155R70J105KA12J" (at 146.05 146.05 0)
+      (effects (font (size 1.27 1.27)) hide)
+    )
     (pin "1")
     (pin "2")
@@
       (effects (font (size 1.27 1.27)) hide)
     )
+    (property "Manufacturer_PN" "RC0402FR-070RL" (at 55.88 144.78 0)
+      (effects (font (size 1.27 1.27)) hide)
+    )
+    (property "Manufacturer" "Yageo" (at 55.88 144.78 0)
+      (effects (font (size 1.27 1.27)) hide)
+    )
     (pin "1")
     (pin "2")
@@
       (effects (font (size 1.27 1.27)) hide)
     )
+    (property "Manufacturer_PN" "RC0402FR-070RL" (at 55.88 167.64 0)
+      (effects (font (size 1.27 1.27)) hide)
+    )
+    (property "Manufacturer" "Yageo" (at 55.88 167.64 0)
+      (effects (font (size 1.27 1.27)) hide)
+    )
     (pin "1")
     (pin "2")
@@
       (effects (font (size 1.27 1.27)) hide)
     )
+    (property "Manufacturer_PN" "RC0402FR-070RL" (at 245.11 124.46 0)
+      (effects (font (size 1.27 1.27)) hide)
+    )
+    (property "Manufacturer" "Yageo" (at 245.11 124.46 0)
+      (effects (font (size 1.27 1.27)) hide)
+    )
     (pin "1")
     (pin "2")
@@
     )
     (property "Datasheet" "~" (at 55.88 152.4 0)
+      (effects (font (size 1.27 1.27)) hide)
+    )
+    (property "Manufacturer_PN" "RC0402FR-070RL" (at 55.88 152.4 0)
+      (effects (font (size 1.27 1.27)) hide)
+    )
+    (property "Manufacturer" "Yageo" (at 55.88 152.4 0)
       (effects (font (size 1.27 1.27)) hide)
     )
@@
       (effects (font (size 1.27 1.27)) hide)
     )
+    (property "Manufacturer_PN" "RC0402FR-070RL" (at 55.88 182.88 0)
+      (effects (font (size 1.27 1.27)) hide)
+    )
+    (property "Manufacturer" "Yageo" (at 55.88 182.88 0)
+      (effects (font (size 1.27 1.27)) hide)
+    )
     (pin "1")
     (pin "2")
@@
       (effects (font (size 1.27 1.27)) hide)
     )
+    (property "Manufacturer_PN" "RC0402FR-070RL" (at 55.88 160.02 0)
+      (effects (font (size 1.27 1.27)) hide)
+    )
+    (property "Manufacturer" "Yageo" (at 55.88 160.02 0)
+      (effects (font (size 1.27 1.27)) hide)
+    )
     (pin "1")
     (pin "2")
@@
       (effects (font (size 1.27 1.27)) hide)
     )
+    (property "Manufacturer_PN" "RC0402FR-070RL" (at 245.11 134.62 0)
+      (effects (font (size 1.27 1.27)) hide)
+    )
+    (property "Manufacturer" "Yageo" (at 245.11 134.62 0)
+      (effects (font (size 1.27 1.27)) hide)
+    )
