File: KiCAD/SZG-SDI-12G-Fire/avr.kicad_sch (KiCad schematic)
At the start: 13 parts, among them J2 Conn_01x06, J3 Conn_02x03_Odd_Even, U1 ATtiny44A-MU

Commit message: Update with part numbers
Add manufacturer part numbers as ordered from DigiKey
Add stitching vias on PCB for SDI 75 ohm striplines

Signed-off-by: Charles Steinkuehler <charles@steinkuehler.net>
Parts:
- C1, C2: Manufacturer (none) -> Murata; Manufacturer_PN (none) -> GRM155R71E104KE14J
- R2: Manufacturer (none) -> Yageo; Manufacturer_PN (none) -> RC0402FR-0710KL
Changed lines of the file:
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@@
+      (effects (font (size 1.27 1.27)) hide)
+    )
+    (property "Manufacturer" "Yageo" (at 124.46 82.55 0)
+      (effects (font (size 1.27 1.27)) hide)
+    )
+    (property "Manufacturer_PN" "RC0402FR-0710KL" (at 124.46 82.55 0)
       (effects (font (size 1.27 1.27)) hide)
     )
@@
       (effects (font (size 1.27 1.27)) hide)
     )
+    (property "Manufacturer" "Murata" (at 85.09 44.45 0)
+      (effects (font (size 1.27 1.27)) hide)
+    )
+    (property "Manufacturer_PN" "GRM155R71E104KE14J" (at 85.09 44.45 0)
+      (effects (font (size 1.27 1.27)) hide)
+    )
     (pin "1")
     (pin "2")
@@
       (effects (font (size 1.27 1.27)) hide)
     )
+    (property "Manufacturer" "Murata" (at 124.46 59.69 0)
+      (effects (font (size 1.27 1.27)) hide)
+    )
+    (property "Manufacturer_PN" "GRM155R71E104KE14J" (at 124.46 59.69 0)
+      (effects (font (size 1.27 1.27)) hide)
+    )
